File: pcb/cooked-tomato.brd (EAGLE design)
At the start: 42 parts, among them IC1 LTC4015, Q1 N_MOSFET_POWERSO8, Q2 N_MOSFET_POWERSO8, Q3 N_MOSFET_POWERSO8

Commit message: Add LTC3300 balancer and LTC6802 monitor schematic
Parts:
- added BRD1: BOARD_STACKINGHWHD_SH, unodex-boards:HWHD_SHARP_CORNERS
- added C23, C25: 1uF, rcl:C0805
- added C24, C26, C28, C29: 0.1uF, rcl:C0603
- added C27: 10uF, rcl:C0805
- added C30, C31, C32, C33, C34, C35: 10uF, rcl:C1206
- added D3: (no value), diode:SOD323-W
- added IC2: LTC6802-1, monitors:SSOP44
- added IC3: LTC3300-1, balancers:LQFP48
- added LED1, LED2, LED3, LED4, LED5, LED6: (no value), led:CHIP-LED0805
- added R11, R12, R13, R14, R15, R16: 220R, rcl:R0603
- added R17, R18, R19, R20: 10K, rcl:R0603
- added R21: 6R8, rcl:R0603
- added X1: STACKING_CONNECTOR_BOTTOM, unodex-boards:HAR-FLEX-BOTTOM-12P
- added X2: STACKING_CONNECTOR_TOP, unodex-boards:HAR-FLEX-TOP-12P
- added X3: (no value), con-molex-micro-fit-3_0:43045-0800
- added X4: (no value), con-molex-micro-fit-3_0:43650-0200
- added X5: (no value), con-molex-micro-fit-3_0:43045-0400
- C21: value 100nF -> 0.1uF
- Q1: value N_MOSFET_POWERSO8 -> (none)
- moved R10 2.43 mm to (16.8, 11.4)
- moved C22 0.82 mm to (14.0, 16.0)
Connections:
- removed net CELL6: IC1.18, IC1.19, R10.2
- removed net NTC: IC1.11, R5.1
- new net +5V: X1.VBUS, X2.VBUS
- new net BAL_CS: IC3.16
- new net BAT_C1: IC2.27, LED6.A, X3.P$7
- new net BAT_C2: IC2.25, LED5.A, X3.P$3
- new net BAT_C3: IC2.23, LED4.A, X3.P$6
- new net BAT_C4: IC2.21, LED3.A, X3.P$2
- new net BAT_C5: IC2.19, LED2.A, X3.P$5
- new net BAT_C6: IC1.18, IC1.19, IC2.11, IC2.13, IC2.15, IC2.17, IC2.4, IC2.5, IC2.7, IC2.9, LED1.A, R10.2, X3.P$1
- new net BAT_NTC: IC1.11, R5.1, X3.P$8
- new net BUS_CLK: X1.CLK, X2.CLK
- new net BUS_DATA: X1.DATA, X2.DATA
- new net BUS_FRAME: X1.FRAME, X2.FRAME
- new net BUS_ID: X1.ID, X2.ID
- new net BUS_IRQ: X1.IRQ, X2.IRQ
- new net BUS_SCL: X1.SCL, X2.SCL
- new net BUS_SDA: X1.SDA, X2.SDA
- new net BUS_WAKEUP: X1.WAKEUP, X2.WAKEUP
- new net G6P: IC3.38
- new net G6S: IC3.1
- new net I6P: IC3.37
- new net I6S: IC3.2
- new net LED_S1: IC2.28, R16.1
- new net LED_S2: IC2.26, R15.1
- new net LED_S3: IC2.24, R14.1
- new net LED_S4: IC2.22, R13.1
- new net LED_S5: IC2.20, R12.1
- new net LED_S6: IC2.18, R11.1
- new net MISO: IC2.43, IC3.19
- new net MON_CS: IC2.44
- new net MOSI: IC2.42, IC3.18
- new net N$20: LED3.C, R13.2
- new net N$21: LED4.C, R14.2
- new net N$25: LED5.C, R15.2
- new net N$26: LED6.C, R16.2
- new net N$27: C25.1, C26.1, IC2.33
- new net N$28: IC3.13, R18.2
- new net N$29: LED1.C, R11.2
- new net N$30: C23.1, C24.1, IC2.34, IC2.35, IC2.36, IC2.40, R17.1
- new net N$31: IC2.37, R17.2
- new net N$32: IC3.14, R19.2
- new net N$33: IC3.20, R20.1
- new net N$34: C27.1, C28.1, IC3.42, IC3.46, IC3.47, IC3.48, R20.2
- new net N$35: C29.2, IC3.41
- new net N$36: C29.1, IC3.40, R21.1
- new net N$37: D3.C, R21.2
- new net N$38: C30.1, D3.A, IC3.39
- new net N$39: C30.2, C31.1, IC3.36
- new net N$40: C31.2, C32.1, IC3.33
- new net N$41: C32.2, C33.1, IC3.30
- new net N$42: C33.2, C34.1, IC3.27
- new net N$43: C34.2, C35.1, IC3.24
- new net N$45: IC3.3
- new net N$46: IC3.4
- new net N$47: IC3.35
- new net N$48: IC3.34
- new net N$49: IC3.5
- new net N$50: IC3.6
- new net N$51: IC3.32
- new net N$52: IC3.31
- new net N$53: IC3.7
- new net N$54: IC3.8
- new net N$55: IC3.29
- new net N$56: IC3.28
- new net N$57: IC3.9
- new net N$58: IC3.10
- new net N$59: IC3.26
- new net N$60: IC3.25
- new net N$61: IC3.11
- new net N$62: IC3.12
- new net N$63: IC3.23
- new net N$64: IC3.22
- new net N$9: LED2.C, R12.2
- new net SCK: IC2.41, IC3.17
- net GND: now also BRD1.HOLE1, BRD1.HOLE2, BRD1.HOLE3, BRD1.HOLE4, C23.2, C24.2, C25.2, C26.2, C27.2, C28.2, C35.2, IC2.29, IC2.30, IC3.15, IC3.21, IC3.PAD, R18.1, R19.1, X1.GND1, X1.GND2, X1.GND3, X1.H1, X1.H2, X1.H3, X1.H4, X2.GND1, X2.GND2, X2.GND3, X2.H1, X2.H2, X2.H3, X2.H4, X3.P$4, X4.P$2
- net VSOLAR: now also X4.P$1
Routing:
- net GND: vias 0 -> 1
- added copper zone on layer 16, net GND
Other:
- board outline added: 50 x 80 mm
