File: pcb/cooked-tomato.sch (EAGLE design)
At the start: 42 parts, among them IC1 LTC4015, Q1 N_MOSFET_POWERSO8, Q2 N_MOSFET_POWERSO8, Q3 N_MOSFET_POWERSO8

Commit message: Add LTC3300 balancer and LTC6802 monitor schematic
Parts:
- added BRD1: BOARD_STACKINGHWHD_SH, unodex-boards:BOARD_STACKINGHWHD_SH
- added C23, C25: 1uF, rcl:C-EUC0805
- added C24, C26, C28, C29: 0.1uF, rcl:C-EUC0603
- added C27: 10uF, rcl:C-EUC0805
- added C30, C31, C32, C33, C34, C35: 10uF, rcl:C-EUC1206
- added D3: (no value), diode:DIODE-SOD323-W
- added IC2: LTC6802-1, monitors:LTC6802-1
- added IC3: LTC3300-1, balancers:LTC3300-1
- added LED1, LED2, LED3, LED4, LED5, LED6: (no value), led:LEDCHIP-LED0805
- added R11, R12, R13, R14, R15, R16: 220R, rcl:R-EU_R0603
- added R17, R18, R19, R20: 10K, rcl:R-EU_R0603
- added R21: 6R8, rcl:R-EU_R0603
- added X1: STACKING_CONNECTOR_BOTTOM, unodex-boards:STACKING_CONNECTOR_BOTTOM
- added X2: STACKING_CONNECTOR_TOP, unodex-boards:STACKING_CONNECTOR_TOP
- added X3: (no value), con-molex-micro-fit-3_0:HEADER_POS8_43045-0800
- added X4: (no value), con-molex-micro-fit-3_0:HEADER_POS2_43650-0200
- added X5: (no value), con-molex-micro-fit-3_0:HEADER_POS4_43045-0401
- C21: value 100nF -> 0.1uF
Connections:
- removed net CELL6: IC1.BATSENS, IC1.CSN, R10.2
- removed net NTC: IC1.NTC, R5.1
- new net +5V: X1.VBUS, X2.VBUS
- new net BAL_CS: IC3.CSBI
- new net BAT_C1: IC2.C1, LED6.A, X3.7
- new net BAT_C2: IC2.C2, LED5.A, X3.3
- new net BAT_C3: IC2.C3, LED4.A, X3.6
- new net BAT_C4: IC2.C4, LED3.A, X3.2
- new net BAT_C5: IC2.C5, LED2.A, X3.5
- new net BAT_C6: IC1.BATSENS, IC1.CSN, IC2.C10, IC2.C11, IC2.C12, IC2.C6, IC2.C7, IC2.C8, IC2.C9, IC2.V+, LED1.A, R10.2, X3.1
- new net BAT_NTC: IC1.NTC, R5.1, X3.8
- new net BUS_CLK: X1.CLK, X2.CLK
- new net BUS_DATA: X1.DATA, X2.DATA
- new net BUS_FRAME: X1.FRAME, X2.FRAME
- new net BUS_ID: X1.ID, X2.ID
- new net BUS_IRQ: X1.IRQ, X2.IRQ
- new net BUS_SCL: X1.SCL, X2.SCL
- new net BUS_SDA: X1.SDA, X2.SDA
- new net BUS_WAKEUP: X1.WAKEUP, X2.WAKEUP
- new net G6P: IC3.G6P
- new net G6S: IC3.G6S
- new net I6P: IC3.I6P
- new net I6S: IC3.I6S
- new net LED_S1: IC2.S1, R16.1
- new net LED_S2: IC2.S2, R15.1
- new net LED_S3: IC2.S3, R14.1
- new net LED_S4: IC2.S4, R13.1
- new net LED_S5: IC2.S5, R12.1
- new net LED_S6: IC2.S6, R11.1
- new net MISO: IC2.SDO, IC3.SDO
- new net MON_CS: IC2.CSBI
- new net MOSI: IC2.SDI, IC3.SDI
- new net N$20: LED3.C, R13.2
- new net N$21: LED4.C, R14.2
- new net N$25: LED5.C, R15.2
- new net N$26: LED6.C, R16.2
- new net N$27: C25.1, C26.1, IC2.VREF
- new net N$28: IC3.RTONS, R18.2
- new net N$29: LED1.C, R11.2
- new net N$30: C23.1, C24.1, IC2.MMB, IC2.TOS, IC2.VMODE, IC2.VREG, R17.1
- new net N$31: IC2.WDTB, R17.2
- new net N$32: IC3.RTONP, R19.2
- new net N$33: IC3.WDT, R20.1
- new net N$34: C27.1, C28.1, IC3.BOOST, IC3.TOS, IC3.VMODE, IC3.VREG, R20.2
- new net N$35: C29.2, IC3.BOOST-
- new net N$36: C29.1, IC3.BOOST+, R21.1
- new net N$37: D3.C, R21.2
- new net N$38: C30.1, D3.A, IC3.C6
- new net N$39: C30.2, C31.1, IC3.C5
- new net N$40: C31.2, C32.1, IC3.C4
- new net N$41: C32.2, C33.1, IC3.C3
- new net N$42: C33.2, C34.1, IC3.C2
- new net N$43: C34.2, C35.1, IC3.C1
- new net N$45: IC3.G5S
- new net N$46: IC3.I5S
- new net N$47: IC3.G5P
- new net N$48: IC3.I5P
- new net N$49: IC3.G4S
- new net N$50: IC3.I4S
- new net N$51: IC3.G4P
- new net N$52: IC3.I4P
- new net N$53: IC3.G3S
- new net N$54: IC3.I3S
- new net N$55: IC3.G3P
- new net N$56: IC3.I3P
- new net N$57: IC3.G2S
- new net N$58: IC3.I2S
- new net N$59: IC3.G2P
- new net N$60: IC3.I2P
- new net N$61: IC3.G1S
- new net N$62: IC3.I1S
- new net N$63: IC3.G1P
- new net N$64: IC3.I1P
- new net N$9: LED2.C, R12.2
- new net SCK: IC2.SCKI, IC3.SCKI
- net GND: now also BRD1.HOLES, C23.2, C24.2, C25.2, C26.2, C27.2, C28.2, C35.2, IC2.NC, IC2.V-, IC3.CTRL, IC3.PAD, IC3.V-, R18.1, R19.1, X1.GND, X2.GND, X3.4, X4.2
- net VSOLAR: now also X4.1
Other:
- note added: "AUX NTC inputs"
- note added: "Balancing indicators"
- note added: "Battery monitor and resistive balancer"
- note added: "Battery pack balancing - power part"
- note added: "Battery pack balancing controller"
- note added: "Battery pack connector"
- note added: "CTRL=V- for multitransformer application"
- note added: "Solar panel connector"
- note added: "upstream port NC"
